File: pcb/easyface485.brd (EAGLE design)
At the start: 89 x 40 mm, 58 parts, among them IC1 MAX487-S, IC2 ATMEGA88-16AU, IC4 PCA9534PW, Q1 MMBT2222, Q2 MMBT2222, U1 L7805D2TT, X2 DG3XX-04-3.5

Commit message: new pcb in progress
Parts:
- moved GND 23.4 mm to (12.0, 44.1), turned to 0 degrees
- moved !RESET 22.1 mm to (10.3, 44.0), turned to 0 degrees
- moved SCK 21.8 mm to (8.20, 44.1), turned to 0 degrees
- moved MOSI 20.5 mm to (4.85, 43.7), turned to 0 degrees
- moved MISO 20.3 mm to (6.53, 43.6), turned to 0 degrees
- moved C10 6.11 mm to (24.4, 28.2)
- moved IC2 4.18 mm to (17.3, 23.6)
- moved R24 2.63 mm to (12.6, 16.2), turned to 270 degrees
- moved Z1 2.37 mm to (21.0, 31.9)
- moved C6 1.67 mm to (29.2, 33.4)
- moved C3 1.61 mm to (29.2, 31.4)
- moved C11 0.55 mm to (9.64, 12.6)
- moved C1 0.51 mm to (8.59, 15.6)
- moved R1 0.45 mm to (10.6, 15.6)
Routing:
- net !RESET: track 31.9 -> 20.4 mm
- net BUZZER: track 19.8 -> 8.81 mm, vias 2 -> 1
- net E: track 78.7 -> 68.1 mm
- net DB1: track 48.3 -> 38.8 mm
- net BL-A: track 56.1 -> 46.9 mm
- net DB0: track 43.5 -> 34.8 mm
- net +5V: track 206.0 -> 197.4 mm, vias 11 -> 10
- net RXD: track 17.9 -> 22.6 mm
- net TXD: track 10.1 -> 14.5 mm
- net N$3: track 6.72 -> 2.52 mm
- net PC2: track 7.45 -> 11.4 mm
- net LIGHT: track 33.8 -> 37.8 mm
- net SCL: track 21.6 -> 25.5 mm
- net SDA: track 15.8 -> 19.8 mm
- net DE: track 12.0 -> 16.0 mm
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